Commit message: modify assets

File: src/mjlab/asset_zoo/robots/walker_s2_hands_v1/urdf/s2_v1.urdf (robot description, URDF)
Before this commit: robot s2_v1, 61 links, 59 joints
Joints:
- removed joint AssemblerFixedJoint
- added joint Left_hands_Joint: type fixed, parent L_sixforce_link, child L_hand_base_link, origin xyz=0.00000004 0.00000001 0.00000001 rpy=0 1.57079601 -0.00000019
- added joint Right_hands_Joint: type fixed, parent R_sixforce_link, child R_hand_base_link, origin xyz=0.00000001 0.00000001 -0.00000001 rpy=0 -1.5707962 3.1415926
